File: Dice.brd (EAGLE design)
At the start: 25.4 x 25.4 mm, 14 parts, among them IC1 PIC12F629SN

Commit message: Always powered
Parts:
- removed SW1: (no value), Seeed-OPL-Switch:SW2-4.0-6.0X3.0X2.5MM
- added SW: (no value), Seeed-OPL-Switch:SW2-4.0-6.0X3.0X2.5MM
- renumbered G1 to BATT
Connections:
- net N$11 renamed LED4
- net N$12 renamed LED2&6
- net N$2 renamed GP0
- net N$3 renamed GP1
- net N$4 renamed GP2
- net N$5 renamed GP4
- net N$6 renamed LED3&5
- net N$7 renamed LED1&7
- removed net N$1: IC1.1, SW1.2
- new net GP3: IC1.4, SW.2
- net VCC: now also IC1.1, SW.1; no longer SW1.1
Routing:
- net VCC: track 10.7 -> 39.7 mm, vias 1 -> 2
- net N$1: track 23.5 -> 0.00 mm, vias 2 -> 0
- net GP3: track 0.00 -> 16.5 mm, vias 0 -> 2
- net GP4: track 8.85 -> 10.1 mm
- net LED3&5: track 35.6 -> 36.2 mm

Commit message: Revision 2
Parts:
- added R5: 47K, resistor:R0805
- R1, R2, R4: value (none) -> 470
- R3: value (none) -> 1K
Connections:
- net GND: now also SW.1
- net GP3: now also R5.1
- net VCC: now also R5.2; no longer SW.1
Routing:
- net VCC: track 39.7 -> 33.0 mm
- net GP3: track 16.5 -> 20.8 mm, vias 2 -> 3
- net LED1&7: track 48.8 -> 46.2 mm
- net GND: track 103.1 -> 104.7 mm, vias 4 -> 2
- net LED3&5: track 36.2 -> 35.6 mm
